Commit message: Update robot description package

File: urdf/robot.urdf (robot description, URDF)
Before this commit: robot techdojo_robot, 5 links, 4 joints
Links:
- link base_link: geometry collision box size=0.3 0.3 0.2; visual box size=0.3 0.3 0.2
Joints:
- joint left_back_wheel_joint: origin xyz=-0.15 0.26 -0.1 rpy=0 0 0 -> xyz=-0.1 0.15 -0.1 rpy=0 0 0
- joint left_front_wheel_joint: origin xyz=0.15 0.26 -0.1 rpy=0 0 0 -> xyz=0.1 0.15 -0.1 rpy=0 0 0
- joint right_back_wheel_joint: origin xyz=-0.15 -0.26 -0.1 rpy=0 0 0 -> xyz=-0.1 -0.15 -0.1 rpy=0 0 0
- joint right_front_wheel_joint: origin xyz=0.15 -0.26 -0.1 rpy=0 0 0 -> xyz=0.1 -0.15 -0.1 rpy=0 0 0

Commit message: Fix indentation in urdf/robot.urdf

File: urdf/robot.urdf (robot description, URDF)
Before this commit: robot techdojo_robot, 5 links, 4 joints
Links:
- added link lidar_link, mass 0.1; collision cylinder length=0.04 radius=0.06; visual mesh filename=package://my_robot_description/meshes/lidar.STL scale=1 1 1
Joints:
- added joint lidar_joint: type fixed, parent base_link, child lidar_link, origin xyz=0 0 0.13 rpy=0 0 0
